File: hw/controller/controller.sch (EAGLE design)
At the start: 105 parts, among them J1 XT30XT30PW_MALE, J2 XT30XT30PW_MALE, M1 MOUNT, M2 MOUNT, M3 MOUNT, M4 MOUNT, Q1 TPH1R204PLSOP_ADVANCE_8, Q2 TPH1R204PLSOP_ADVANCE_8, Q3 TPH1R204PLSOP_ADVANCE_8, Q4 TPH1R204PLSOP_ADVANCE_8, Q5 TPH1R204PLSOP_ADVANCE_8, Q6 TPH1R204PLSOP_ADVANCE_8, U1 STM32G474CEU6, U2 TCAN334GSOT23, U3 AS5147, U4 DRV8323RS

Commit message: Initial work on r4.5
Parts:
- A, B, C: value PAD -> PAD16AWG_PAD; device controller:PAD -> controller:PAD16AWG_PAD
- Q1, Q2, Q3, Q4, Q5, Q6: MPN TPH1R204PL,L1Q -> TPH2R506PL,L1Q
- R6: value 10k 1% -> 4.7k 1%; MPN ERJ-2RKF1002X -> ERJ-2RKF4701X
Connections:
- net GND: now also U1.PA15; no longer U1.PC6
Other:
- note added: "PC13/PA15/PC6 Version 101"
- note added: "moteus r4.5 (c) jjp@pobox.com 2019 Licensed under the Apache 2.0 License"
- note removed: "PC13/PA15/PC6 Version 110"
- note removed: "moteus r4.4 (c) jjp@pobox.com 2019 Licensed under the Apache 2.0 License"
Changed lines of the file:
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@@
 <attribute name="MPN" value="ERJ-2RKF1003X"/>
 </part>
-<part name="R6" library="mfpassives" deviceset="RESISTOR" device="_0402" value="10k 1%">
+<part name="R6" library="mfpassives" deviceset="RESISTOR" device="_0402" value="4.7k 1%">
 <attribute name="MF" value="Panasonic"/>
-<attribute name="MPN" value="ERJ-2RKF1002X"/>
+<attribute name="MPN" value="ERJ-2RKF4701X"/>
 </part>
 <part name="U3" library="controller" deviceset="AS5147" device="">
@@
 <part name="Q1" library="controller" deviceset="TPH1R204PL" device="SOP_ADVANCE_8">
 <attribute name="MF" value="Toshiba"/>
-<attribute name="MPN" value="TPH1R204PL,L1Q"/>
+<attribute name="MPN" value="TPH2R506PL,L1Q"/>
 <attribute name="POPULATE" value="1"/>
 </part>
 <part name="Q2" library="controller" deviceset="TPH1R204PL" device="SOP_ADVANCE_8">
 <attribute name="MF" value="Toshiba"/>
-<attribute name="MPN" value="TPH1R204PL,L1Q"/>
+<attribute name="MPN" value="TPH2R506PL,L1Q"/>
 <attribute name="POPULATE" value="1"/>
 </part>
 <part name="Q3" library="controller" deviceset="TPH1R204PL" device="SOP_ADVANCE_8">
 <attribute name="MF" value="Toshiba"/>
-<attribute name="MPN" value="TPH1R204PL,L1Q"/>
+<attribute name="MPN" value="TPH2R506PL,L1Q"/>
 <attribute name="POPULATE" value="1"/>
 </part>
 <part name="Q4" library="controller" deviceset="TPH1R204PL" device="SOP_ADVANCE_8">
 <attribute name="MF" value="Toshiba"/>
-<attribute name="MPN" value="TPH1R204PL,L1Q"/>
+<attribute name="MPN" value="TPH2R506PL,L1Q"/>
 <attribute name="POPULATE" value="1"/>
 </part>
 <part name="Q5" library="controller" deviceset="TPH1R204PL" device="SOP_ADVANCE_8">
 <attribute name="MF" value="Toshiba"/>
-<attribute name="MPN" value="TPH1R204PL,L1Q"/>
+<attribute name="MPN" value="TPH2R506PL,L1Q"/>
 <attribute name="POPULATE" value="1"/>
 </part>
 <part name="Q6" library="controller" deviceset="TPH1R204PL" device="SOP_ADVANCE_8">
 <attribute name="MF" value="Toshiba"/>
-<attribute name="MPN" value="TPH1R204PL,L1Q"/>
+<attribute name="MPN" value="TPH2R506PL,L1Q"/>
 <attribute name="POPULATE" value="1"/>
 </part>
@@
 <attribute name="MPN" value="CGA2B3X7R1H104K050BB"/>
 </part>
-<part name="A" library="controller" deviceset="PAD" device="">
-<attribute name="POPULATE" value="0"/>
-</part>
-<part name="B" library="controller" deviceset="PAD" device="">
-<attribute name="POPULATE" value="0"/>
-</part>
-<part name="C" library="controller" deviceset="PAD" device="">
+<part name="A" library="controller" deviceset="PAD" device="16AWG_PAD" value="PAD16AWG_PAD">
+<attribute name="POPULATE" value="0"/>
+</part>
+<part name="B" library="controller" deviceset="PAD" device="16AWG_PAD" value="PAD16AWG_PAD">
+<attribute name="POPULATE" value="0"/>
+</part>
+<part name="C" library="controller" deviceset="PAD" device="16AWG_PAD" value="PAD16AWG_PAD">
 <attribute name="POPULATE" value="0"/>
 </part>
@@
 <text x="-132.08" y="-142.24" size="5.08" layer="90">POWER FETS</text>
 <text x="73.66" y="-142.24" size="5.08" layer="90">BULK CAPACITANCE</text>
-<text x="-307.34" y="200.66" size="7.62" layer="90">moteus r4.4
+<text x="-307.34" y="200.66" size="7.62" layer="90">moteus r4.5
 (c) jjp@pobox.com 2019
 Licensed under the Apache 2.0 License</text>
 <text x="22.86" y="111.76" size="1.778" layer="91">PC13/PA15/PC6 Version
-110</text>
+101</text>
 </plain>
 <instances>
@@
 <attribute name="VALUE" x="-292.1" y="-238.76" size="1.778" layer="96" rot="R90"/>
 </instance>
-<instance part="GND22" gate="1" x="30.48" y="96.52" smashed="yes">
-<attribute name="VALUE" x="27.94" y="93.98" size="1.778" layer="96"/>
+<instance part="GND22" gate="1" x="20.32" y="147.32" smashed="yes">
+<attribute name="VALUE" x="17.78" y="144.78" size="1.778" layer="96"/>
 </instance>
 </instances>
@@
 </segment>
 <segment>
-<pinref part="U1" gate="G$1" pin="PC6"/>
-<wire x1="-22.86" y1="104.14" x2="30.48" y2="104.14" width="0.1524" layer="91"/>
-<wire x1="30.48" y1="104.14" x2="30.48" y2="99.06" width="0.1524" layer="91"/>
+<pinref part="U1" gate="G$1" pin="PA15"/>
+<wire x1="-33.02" y1="144.78" x2="-33.02" y2="154.94" width="0.1524" layer="91"/>
+<wire x1="-33.02" y1="154.94" x2="20.32" y2="154.94" width="0.1524" layer="91"/>
 <pinref part="GND22" gate="1" pin="GND"/>
+<wire x1="20.32" y1="154.94" x2="20.32" y2="149.86" width="0.1524" layer="91"/>
 </segment>
 </net>
