File: hw/power_dist/power_dist.sch (EAGLE design)
At the start: 57 parts, among them J1 JST-ZH6SMT_VERT, J2 JST-PH4SMT_VERT, P1 XT30P, P2 XT30P, P3 XT30P, P4 XT30P, P5 XT30P, P6 XT30P, P7 XT90PW-M, Q1 TPH1R204PL, Q2 TPH1R204PL, Q3 TPH1R204PL, U1 ZXTR2012Z, U2 MAX150628TDFN, U3 STM32G474CEU6, U4 MIC4416, U5 MIC4416, U6 TCAN334G

Commit message: WIP of power_dist r4
Parts:
- removed D12, D3V3, DG, DI: PAD24AWG_PAD, precharge:PAD24AWG_PAD
- removed D2: (no value), mfleds:LED_SINGLE-0603
- removed D3: (no value), imu_junction:DIODE-
- removed Q1, Q2, Q3: TPH1R204PL, imu_junction:TPH1R204PL
- added CR1: SMBJ51CA-E3/52, power_dist:SMBJ51CA-E3/52
- added MOSFET1, MOSFET2, MOSFET3: PSMN4R8-100BSEJ, power_dist:PSMN4R8-100BSEJ
- added R11, R12: 10k, mfpassives:RESISTOR_0603
- added R13: 15k 1%, mfpassives:RESISTOR_0603
- added U$5: JST-PH5VERT, power_dist:JST-PH5VERT
- added U7: MF-DSC-SOT233-BSS138, mfdiscretesemi:N-CHANNEL_FET_BSS138_SOT-23-3
- C1: value 1uF 50V -> 1uF; HOUSEPART (none) -> 1; MF SAMSUNG -> (none); MPN CL10A105KB8NNNC -> MF-CAP-0603-1uF
- C10, C11, C12, C13, C3, C4: device mfpassives:CAPACITOR_NP_0402 -> mfpassives:CAPACITOR_NP_0603; MPN MF-CAP-0402-0.1uF -> MF-CAP-0603-0.1uF
- C14: device mfpassives:CAPACITOR_NP_0402 -> mfpassives:CAPACITOR_NP_0603; MPN MF-CAP-0402-1uF -> MF-CAP-0603-1uF
- C5: value 0.1uF -> 0.01uF; device mfpassives:CAPACITOR_NP_0402 -> mfpassives:CAPACITOR_NP_0603; MPN MF-CAP-0402-0.1uF -> MF-CAP-0603-0.01uF
- C6: value 0.1uF -> 0.082uF; device mfpassives:CAPACITOR_NP_0402 -> mfpassives:CAPACITOR_NP_0603; HOUSEPART 1 -> 0; MF (none) -> YAGEO; MPN MF-CAP-0402-0.1uF -> CC0603KRX7R9BB823
- C7: value 10uF 50V -> 1uF; device mfpassives:CAPACITOR_NP_1206 -> mfpassives:CAPACITOR_NP_0603; HOUSEPART (none) -> 1; MF TDK -> (none); MPN C3216X7R1H106K160AE -> MF-CAP-0603-1uF
- C8, C9: value 1uF 50V -> 1uF 100V; device mfpassives:CAPACITOR_NP_0603 -> mfpassives:CAPACITOR_NP_0805; MF SAMSUNG -> MURATA; MPN CL10A105KB8NNNC -> GCM21BC72A105KE36L
- D1: value (none) -> MF-DIO-SOD123-1N4148; device mfleds:LED_SINGLE-0603 -> mfdiscretesemi:DIODES_1N4148_SOD-123; HOUSEPART 1 -> (none); MPN MF-LED-0603-RED -> (none)
- L1: value 33uH -> CBC3225T330KR; device mfpassives:INDUCTOR_1210 -> power_dist:CBC3225T330KR; MF TDK -> (none); MPN NLFV32T-330K-EF -> CBC3225T330KR
- R1: value 220 -> 47k 1%; HOUSEPART 1 -> (none); MPN MF-RES-0603-220 -> (none)
- R2: value 220 -> 15k 1%; HOUSEPART 1 -> (none); MPN MF-RES-0603-220 -> (none)
- R3: MF VISHAY -> (none); MPN CRCW0603100KFKEA -> (none)
- R4: value 10k 1% -> 4.7k 1%; MF PANASONIC -> (none); MPN ERJ-3EKF1002V -> (none)
- R5: value 100k 1% -> 0.3mOhm; device mfpassives:RESISTOR_0603 -> power_dist:SENSE_RESISTOR2512; MF VISHAY -> VISHAY DALE; MPN CRCW0603100KFKEA -> WSLF2512L3000FEA; POPULATE (none) -> 1
- R6: value 10k 1% -> 24k 1%; MF PANASONIC -> (none); MPN ERJ-3EKF1002V -> (none)
- R7: value 10 1W -> 1k 1%; device mfpassives:RESISTOR_1206 -> mfpassives:RESISTOR_0603; MF Susumu -> (none); MPN HRG3216Q-10R0-D-T1 -> (none)
- R8: value 100k 1% -> 10k; HOUSEPART (none) -> 1; MF VISHAY -> (none); MPN CRCW0603100KFKEA -> MF-RES-0603-10K
- R9: value 100k 1% -> 47k 1%; MF VISHAY -> (none); MPN CRCW0603100KFKEA -> (none)
- U1: value ZXTR2012Z -> MAX15062AATA+T; device imu_junction:ZXTR2012Z -> power_dist:MAX15062AATA+T; MPN ZXTR2012Z-13 -> MAX15062AATA+T; POPULATE (none) -> 1
- U2: value MAX150628TDFN -> LM5066IPMHE/NOPB; device precharge:MAX150628TDFN -> power_dist:LM5066IPMHE/NOPB; MF MAXIM -> (none); MPN MAX15062AATA+T -> (none); POPULATE 1 -> (none)
- U4: value MIC4416 -> FSV10150V; device imu_junction:MIC4416 -> power_dist:FSV10150V; MPN (none) -> FSV10150V; POPULATE (none) -> 1
- U5: value MIC4416 -> MF-DSC-SOT233-MMBT3906; device imu_junction:MIC4416 -> mfdiscretesemi:PNP_BJT_MMBT3906_SOT-23-3
Connections:
- removed net +12V: C2.P$1, C5.P$1, C6.P$1, D12.P$1, U1.VOUT, U4.VS, U5.VS
- removed net +18V: C1.P$1, C8.P$1, D3.C, DI.P$1, P1.2, P2.2, P3.2, P4.2, P5.2, P6.2, P7.2, R3.P$2, U1.VIN, U2.EN, U2.VIN
- removed net FET_MAIN: R9.P$2, U3.PA1, U5.CTL
- removed net FET_PRECHARGE: R8.P$2, U3.PA0, U4.CTL
- removed net LX: L1.P$1, U2.LX
- removed net PCHG: Q1.D, R7.P$1
- removed net V-OUT: D3.A, P1.1, P2.1, P3.1, P4.1, P5.1, P6.1, Q2.D, Q3.D, R5.P$2, R7.P$2
- removed net VSAMP_IN: R3.P$1, R4.P$2, U3.PA9
- removed net VSAMP_OUT: R5.P$1, R6.P$2, U3.PA8
- new net +24V: C8.P$1, CR1.1, P7.2, R1.P$1, R3.P$1, R5.1, R9.P$1, U1.EN/UVLO, U1.VIN, U2.VIN
- new net GPIO1: U$5.4, U3.PC10
- new net GPIO2: U$5.3, U3.PC11
- new net GPIO3: U$5.2, U3.PB3
- new net N$10: R6.P$1, U2.PWR
- new net N$11: C5.P$1, U2.TIMER
- new net N$5: D1.ANODE, MOSFET1.G, MOSFET2.G, MOSFET3.G, R7.P$1, U2.GATE
- new net N$6: C7.P$1, U2.VDD
- new net N$9: R1.P$2, R2.P$1, U2.UVLO/EN, U7.DRAIN
- new net PSHDN: R13.P$1, R9.P$2, U3.PB13, U7.GATE
- new net SCL: R11.P$1, U2.SCL, U3.PA9
- new net SDA: R8.P$1, U2.SDAI, U2.SDAO, U3.PA8
- new net SMBA: R12.P$1, U2.!SMBA, U3.PA10
- new net VIN_SENSE: R3.P$2, R4.P$1, U2.OVLO
- new net VSENSE_HIGH: R5.S1, U2.VIN_K
- new net VSENSE_LOW: R5.S2, U2.SENSE
- new net VSWITCHED: C9.P$1, MOSFET1.S, MOSFET2.S, MOSFET3.S, P1.2, P2.2, P3.2, P4.2, P5.2, P6.2, U2.OUT, U4.CATHODE
- net CAN_SHDN: now also U3.PB14; no longer U3.PA10
- net GND: now also CR1.2, P1.1, P2.1, P3.1, P4.1, P5.1, P6.1, R13.P$2, R2.P$2, R4.P$2, R6.P$2, R7.P$2, U$5.5, U2.AGND, U4.ANODE, U4.ANODE_2, U5.BASE, U7.SOURCE; no longer DG.P$1, Q1.S, Q2.S, Q3.S, R4.P$1, R6.P$1, R8.P$1, R9.P$1, U4.GND, U5.GND
- net LED1: no longer D1.CATHODE
- net LED2: no longer D2.CATHODE
- net N$1: now also L1.2, U1.LX; no longer D1.ANODE, R1.P$1
- net N$12: now also C6.P$1, U5.EMITTER; no longer Q1.G, U4.G
- net N$13: now also D1.CATHODE, U5.COLLECTOR; no longer C9.P$1, U2.VCC
- net N$3: now also MOSFET1.D, MOSFET2.D, MOSFET3.D, R5.2; no longer Q2.G, Q3.G, U5.G
- net N$4: now also C1.P$1, U1.VCC; no longer D2.ANODE, R2.P$1
- net VCC: now also C2.P$1, L1.1, R11.P$2, R12.P$2, R8.P$2, U$5.1, U1.FB/VOUT; no longer C7.P$1, D3V3.P$1, L1.P$2, R1.P$2, R2.P$2, U2.FB
Other:
- note added: "Min / Typ / Max Upper UVLO: 10.69 / 11.32 / 11.95 Lower UVLO: 10.13 / 10.33 / 10.54 Upper OVLO: 54.58 / 55.69 / 56.81 Lower OVLO: 51.58 / 53.59 / 55.61"
- note added: "mjbots power dist r4.0 (c) 2020 Josh Pieper, jjp@pobox.com Licensed under the Apache 2.0 License https://www.apache.org/licenses/LICENSE-2.0"
- note removed: "mjbots power dist r3.1 (c) 2020 Josh Pieper, jjp@pobox.com Licensed under the Apache 2.0 License https://www.apache.org/licenses/LICENSE-2.0"
- moved on the sheet: C1, C2, C5, C6, C7, C8, C9, R1, R2, R3, R4, R6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

Commit message: power_dist r4 rough layout and most things renumbered
Parts:
- removed CR1: SMBJ51CA-E3/52, power_dist:SMBJ51CA-E3/52
- removed U6: TCAN334G, precharge:TCAN334G
- added C16: 0.1uF, mfpassives:CAPACITOR_NP_0603
- added D2: MF-DIO-SOD123-1N4148, mfdiscretesemi:DIODES_1N4148_SOD-123
- added D3: FSV10150V, power_dist:FSV10150V
- added DB_3, DB_G, DB_VIN, DB_VSW: PAD24AWG_PAD, precharge:PAD24AWG_PAD
- C1: value 1uF -> 1uF 100V; device mfpassives:CAPACITOR_NP_0603 -> mfpassives:CAPACITOR_NP_0805; HOUSEPART 1 -> (none); MF (none) -> MURATA; MPN MF-CAP-0603-1uF -> GCM21BC72A105KE36L
- C11, C12: value 0.1uF -> 1uF; MPN MF-CAP-0603-0.1uF -> MF-CAP-0603-1uF
- C13: value 0.1uF -> 0.01uF; MPN MF-CAP-0603-0.1uF -> MF-CAP-0603-0.01uF
- C14: value 1uF -> 0.01uF; MPN MF-CAP-0603-1uF -> MF-CAP-0603-0.01uF
- C15: value 10uF 50V -> 1uF 100V; device mfpassives:CAPACITOR_NP_1206 -> mfpassives:CAPACITOR_NP_0805; MF TDK -> MURATA; MPN C3216X7R1H106K160AE -> GCM21BC72A105KE36L
- C2: value 10uF 50V -> 1uF; device mfpassives:CAPACITOR_NP_1206 -> mfpassives:CAPACITOR_NP_0603; HOUSEPART (none) -> 1; MF TDK -> (none); MPN C3216X7R1H106K160AE -> MF-CAP-0603-1uF
- C3: value 0.1uF -> 10uF 50V; device mfpassives:CAPACITOR_NP_0603 -> mfpassives:CAPACITOR_NP_1206; HOUSEPART 1 -> (none); MF (none) -> TDK; MPN MF-CAP-0603-0.1uF -> C3216X7R1H106K160AE
- C5: value 0.01uF -> 0.1uF; MPN MF-CAP-0603-0.01uF -> MF-CAP-0603-0.1uF
- C6: value 0.082uF -> 1uF; HOUSEPART 0 -> 1; MF YAGEO -> (none); MPN CC0603KRX7R9BB823 -> MF-CAP-0603-1uF
- C7: value 1uF -> 0.1uF; MPN MF-CAP-0603-1uF -> MF-CAP-0603-0.1uF
- C8: value 1uF 100V -> 0.1uF; device mfpassives:CAPACITOR_NP_0805 -> mfpassives:CAPACITOR_NP_0603; HOUSEPART (none) -> 1; MF MURATA -> (none); MPN GCM21BC72A105KE36L -> MF-CAP-0603-0.1uF
- C9: value 1uF 100V -> 10uF 50V; device mfpassives:CAPACITOR_NP_0805 -> mfpassives:CAPACITOR_NP_1206; MF MURATA -> TDK; MPN GCM21BC72A105KE36L -> C3216X7R1H106K160AE
- D1: value MF-DIO-SOD123-1N4148 -> SMBJ51CA-E3/52; device mfdiscretesemi:DIODES_1N4148_SOD-123 -> power_dist:SMBJ51CA-E3/52; MPN (none) -> SMBJ51CA-E3/52; POPULATE (none) -> 1
- R1: value 47k 1% -> 10k; HOUSEPART (none) -> 1; MPN (none) -> MF-RES-0603-10K
- R10: value 220 -> 0.3mOhm; device mfpassives:RESISTOR_0603 -> power_dist:SENSE_RESISTOR2512; HOUSEPART 1 -> (none); MF (none) -> VISHAY DALE; MPN MF-RES-0603-220 -> WSLF2512L3000FEA; POPULATE (none) -> 1
- R11: value 10k -> 24k 1%; HOUSEPART 1 -> (none); MPN MF-RES-0603-10K -> (none)
- R12: value 10k -> 1k 1%; HOUSEPART 1 -> (none); MPN MF-RES-0603-10K -> (none)
- R13: value 15k 1% -> 220; HOUSEPART (none) -> 1; MPN (none) -> MF-RES-0603-220
- R2: value 15k 1% -> 10k; HOUSEPART (none) -> 1; MPN (none) -> MF-RES-0603-10K
- R3: value 100k 1% -> 10k; HOUSEPART (none) -> 1; MPN (none) -> MF-RES-0603-10K
- R4: value 4.7k 1% -> 47k 1%
- R5: value 0.3mOhm -> 15k 1%; device power_dist:SENSE_RESISTOR2512 -> mfpassives:RESISTOR_0603; MF VISHAY DALE -> (none); MPN WSLF2512L3000FEA -> (none); POPULATE 1 -> (none)
- R6: value 24k 1% -> 47k 1%
- R7: value 1k 1% -> 19.1k 1%
- R8: value 10k -> 140k 1%; HOUSEPART 1 -> (none); MPN MF-RES-0603-10K -> (none)
- R9: value 47k 1% -> 6.49k 1%
- U2: value LM5066IPMHE/NOPB -> STM32G474CEU6; device power_dist:LM5066IPMHE/NOPB -> precharge:STM32G474CEU6; MF (none) -> ST; MPN (none) -> STM32G474CEU6; POPULATE (none) -> 1
- U3: value STM32G474CEU6 -> LM5066IPMHE/NOPB; device precharge:STM32G474CEU6 -> power_dist:LM5066IPMHE/NOPB; MF ST -> (none); MPN STM32G474CEU6 -> (none); POPULATE 1 -> (none)
- U4: value FSV10150V -> TCAN334G; device power_dist:FSV10150V -> precharge:TCAN334G; MF (none) -> Analog; MPN FSV10150V -> LTC2875IS8
- renumbered MOSFET1 to Q1, MOSFET2 to Q2, MOSFET3 to Q3, U$5 to J3, U5 to Q5, U7 to Q4
Connections:
- new net N$7: C11.P$1, U3.VREF
- net +24V: now also C1.P$1, D1.1, DB_VIN.P$1, R10.1, R4.P$1, R6.P$1, R8.P$1, U3.VIN; no longer C8.P$1, CR1.1, R1.P$1, R3.P$1, R5.1, R9.P$1, U2.VIN
- net CAN_N: now also U4.CANL; no longer U6.CANL
- net CAN_P: now also U4.CANH; no longer U6.CANH
- net CAN_RX: now also U2.PA11, U4.RXD; no longer U3.PA11, U6.RXD
- net CAN_SHDN: now also U2.PB14, U4.SHDN; no longer U3.PB14, U6.SHDN
- net CAN_TX: now also U2.PA12, U4.TXD; no longer U3.PA12, U6.TXD
- net GND: now also C16.P$2, D1.2, D3.ANODE, D3.ANODE_2, DB_G.P$1, R11.P$2, R12.P$2, R5.P$2, R9.P$2, U2.PC6, U2.THERMALPAD, U3.AGND, U3.GND, U4.GND, U4.STB; no longer CR1.2, R13.P$2, R2.P$2, R4.P$2, R6.P$2, U2.AGND, U2.GND, U3.THERMALPAD, U4.ANODE, U4.ANODE_2, U6.GND, U6.STB
- net GPIO1: now also U2.PC10; no longer U3.PC10
- net GPIO2: now also U2.PC11; no longer U3.PC11
- net GPIO3: now also U2.PB3; no longer U3.PB3
- net LED1: now also U2.PB9; no longer U3.PB9
- net LED2: now also U2.PB7; no longer U3.PB7
- net N$10: now also R11.P$1, U3.PWR; no longer R6.P$1, U2.PWR
- net N$11: now also C13.P$1, U3.TIMER; no longer C5.P$1, U2.TIMER
- net N$12: now also C14.P$1; no longer C6.P$1
- net N$13: now also D2.CATHODE; no longer D1.CATHODE
- net N$2: now also R13.P$1; no longer R10.P$1
- net N$3: now also R10.2; no longer R5.2
- net N$4: now also C2.P$1; no longer C1.P$1
- net N$5: now also D2.ANODE, R12.P$1, U3.GATE; no longer D1.ANODE, R7.P$1, U2.GATE
- net N$6: now also C12.P$1, U3.VDD; no longer C7.P$1, U2.VDD
- net N$9: now also R6.P$2, R7.P$1, U3.UVLO/EN; no longer R1.P$2, R2.P$1, U2.UVLO/EN
- net NRST: now also C4.P$1, U2.PG10-NRST; no longer C3.P$1, U3.PG10-NRST
- net PSHDN: now also R4.P$2, R5.P$1, U2.PB13; no longer R13.P$1, R9.P$2, U3.PB13
- net PWR_LED: now also U2.PA2; no longer U3.PA2
- net PWR_SW: now also U2.PA3; no longer U3.PA3
- net SCL: now also R2.P$1, U2.PA9, U3.SCL; no longer R11.P$1, U2.SCL, U3.PA9
- net SDA: now also R1.P$1, U2.PA8, U3.SDAI, U3.SDAO; no longer R8.P$1, U2.SDAI, U2.SDAO, U3.PA8
- net SMBA: now also R3.P$1, U2.PA10, U3.!SMBA; no longer R12.P$1, U2.!SMBA, U3.PA10
- net SWCLK: now also U2.PA14; no longer U3.PA14
- net SWDIO: now also U2.PA13; no longer U3.PA13
- net VCC: now also C16.P$1, C3.P$1, C5.P$1, C6.P$1, C7.P$1, C8.P$1, C9.P$1, DB_3.P$1, R1.P$2, R13.P$2, R2.P$2, R3.P$2, U2.VBAT, U2.VDDA, U2.VDD_1, U2.VDD_2, U2.VDD_3, U2.VREF+, U4.VCC; no longer C11.P$1, C12.P$1, C13.P$1, C14.P$1, C15.P$1, C2.P$1, C4.P$1, R10.P$2, R11.P$2, R12.P$2, R8.P$2, U3.VBAT, U3.VDDA, U3.VDD_1, U3.VDD_2, U3.VDD_3, U3.VREF+, U6.VCC
- net VIN_SENSE: now also R8.P$2, R9.P$1, U3.OVLO; no longer R3.P$2, R4.P$1, U2.OVLO
- net VSENSE_HIGH: now also R10.S1, U3.VIN_K; no longer R5.S1, U2.VIN_K
- net VSENSE_LOW: now also R10.S2, U3.SENSE; no longer R5.S2, U2.SENSE
- net VSWITCHED: now also C15.P$1, D3.CATHODE, DB_VSW.P$1, U3.OUT; no longer C9.P$1, U2.OUT, U4.CATHODE
Other:
- note added: "Min / Typ / Max Upper UVLO: 9.95 Lower UVLO: 8.82 Upper OVLO: 57.11 Lower OVLO: 54.87"
- note added: "PC13/PA15/PC6 Version 110"
- note removed: "Min / Typ / Max Upper UVLO: 10.69 / 11.32 / 11.95 Lower UVLO: 10.13 / 10.33 / 10.54 Upper OVLO: 54.58 / 55.69 / 56.81 Lower OVLO: 51.58 / 53.59 / 55.61"
- moved on the sheet: C1, C10, C11, C12, C13, C14, C15, C2, C3, C4, C5, C6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

Commit message: WIP checkpoint of power_dist r4
Parts:
- added D4, D5: (no value), mfleds:LED_SINGLE-0603
- added R14, R15: 220, mfpassives:RESISTOR_0603
Connections:
- new net N$14: D5.ANODE, R15.P$1
- new net N$8: D4.ANODE, R14.P$1
- net LED1: now also D4.CATHODE, U2.PA0; no longer U2.PB9
- net LED2: now also D5.CATHODE, U2.PA1; no longer U2.PB7
- net VCC: now also R14.P$2, R15.P$2
Changed lines of the file:
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@@
 <part name="P+10" library="supply1" deviceset="VCC" device=""/>
 <part name="P+11" library="supply1" library_urn="urn:adsk.eagle:library:371" deviceset="+24V" device=""/>
+<part name="D4" library="mfleds" deviceset="LED_SINGLE" device="-0603">
+<attribute name="HOUSEPART" value="1"/>
+<attribute name="MPN" value="MF-LED-0603-RED"/>
+</part>
+<part name="R14" library="mfpassives" deviceset="RESISTOR" device="_0603" value="220">
+<attribute name="HOUSEPART" value="1"/>
+<attribute name="MPN" value="MF-RES-0603-220"/>
+</part>
+<part name="P+12" library="supply1" deviceset="VCC" device=""/>
+<part name="D5" library="mfleds" deviceset="LED_SINGLE" device="-0603">
+<attribute name="HOUSEPART" value="1"/>
+<attribute name="MPN" value="MF-LED-0603-RED"/>
+</part>
+<part name="R15" library="mfpassives" deviceset="RESISTOR" device="_0603" value="220">
+<attribute name="HOUSEPART" value="1"/>
+<attribute name="MPN" value="MF-RES-0603-220"/>
+</part>
+<part name="P+13" library="supply1" deviceset="VCC" device=""/>
 </parts>
 <sheets>
@@
 <attribute name="VALUE" x="259.08" y="-7.62" size="1.778" layer="96" rot="R90"/>
 </instance>
+<instance part="D4" gate="G$1" x="200.66" y="-35.56" smashed="yes" rot="R270">
+<attribute name="NAME" x="198.12" y="-33.02" size="1.016" layer="95" font="vector" rot="R270" align="top-left"/>
+<attribute name="VALUE" x="195.58" y="-33.02" size="1.016" layer="96" font="vector" rot="R270"/>
+</instance>
+<instance part="R14" gate="G$1" x="200.66" y="-25.4" smashed="yes" rot="R180">
+<attribute name="NAME" x="198.12" y="-26.924" size="1.016" layer="95" font="vector" rot="R180" align="top-left"/>
+<attribute name="VALUE" x="198.12" y="-23.876" size="1.016" layer="96" font="vector" rot="R180"/>
+</instance>
+<instance part="P+12" gate="VCC" x="200.66" y="-15.24" smashed="yes">
+<attribute name="VALUE" x="198.12" y="-17.78" size="1.778" layer="96" rot="R90"/>
+</instance>
+<instance part="D5" gate="G$1" x="208.28" y="-35.56" smashed="yes" rot="R270">
+<attribute name="NAME" x="205.74" y="-33.02" size="1.016" layer="95" font="vector" rot="R270" align="top-left"/>
+<attribute name="VALUE" x="203.2" y="-33.02" size="1.016" layer="96" font="vector" rot="R270"/>
+</instance>
+<instance part="R15" gate="G$1" x="208.28" y="-25.4" smashed="yes" rot="R180">
+<attribute name="NAME" x="205.74" y="-26.924" size="1.016" layer="95" font="vector" rot="R180" align="top-left"/>
+<attribute name="VALUE" x="205.74" y="-23.876" size="1.016" layer="96" font="vector" rot="R180"/>
+</instance>
+<instance part="P+13" gate="VCC" x="208.28" y="-15.24" smashed="yes">
+<attribute name="VALUE" x="205.74" y="-17.78" size="1.778" layer="96" rot="R90"/>
+</instance>
 </instances>
 <busses>
@@
 <wire x1="259.08" y1="-35.56" x2="271.78" y2="-35.56" width="0.1524" layer="91"/>
 </segment>
+<segment>
+<pinref part="R14" gate="G$1" pin="P$2"/>
+<pinref part="P+12" gate="VCC" pin="VCC"/>
+<wire x1="200.66" y1="-20.32" x2="200.66" y2="-17.78" width="0.1524" layer="91"/>
+</segment>
+<segment>
+<pinref part="R15" gate="G$1" pin="P$2"/>
+<pinref part="P+13" gate="VCC" pin="VCC"/>
+<wire x1="208.28" y1="-20.32" x2="208.28" y2="-17.78" width="0.1524" layer="91"/>
+</segment>
 </net>
 <net name="NRST" class="0">
@@
 <net name="LED1" class="0">
 <segment>
-<pinref part="U2" gate="G$1" pin="PB9"/>
-<wire x1="459.74" y1="175.26" x2="459.74" y2="187.96" width="0.1524" layer="91"/>
-<label x="459.74" y="182.88" size="1.778" layer="95" rot="R90"/>
+<pinref part="D4" gate="G$1" pin="CATHODE"/>
+<wire x1="200.66" y1="-38.1" x2="200.66" y2="-53.34" width="0.1524" layer="91"/>
+<label x="198.12" y="-53.34" size="1.778" layer="95" font="vector" rot="R90"/>
+</segment>
+<segment>
+<pinref part="U2" gate="G$1" pin="PA0"/>
+<wire x1="447.04" y1="134.62" x2="421.64" y2="134.62" width="0.1524" layer="91"/>
+<label x="421.64" y="134.62" size="1.778" layer="95"/>
 </segment>
 </net>
@@
 <net name="LED2" class="0">
 <segment>
-<pinref part="U2" gate="G$1" pin="PB7"/>
-<wire x1="464.82" y1="175.26" x2="464.82" y2="187.96" width="0.1524" layer="91"/>
-<label x="464.82" y="182.88" size="1.778" layer="95" rot="R90"/>
+<pinref part="D5" gate="G$1" pin="CATHODE"/>
+<wire x1="208.28" y1="-38.1" x2="208.28" y2="-53.34" width="0.1524" layer="91"/>
+<label x="208.28" y="-53.34" size="1.778" layer="95" font="vector" rot="R90"/>
+</segment>
+<segment>
+<pinref part="U2" gate="G$1" pin="PA1"/>
+<wire x1="447.04" y1="132.08" x2="421.64" y2="132.08" width="0.1524" layer="91"/>
+<label x="421.64" y="132.08" size="1.778" layer="95"/>
 </segment>
 </net>
@@
 </segment>
 </net>
+<net name="N$8" class="0">
+<segment>
+<pinref part="R14" gate="G$1" pin="P$1"/>
+<pinref part="D4" gate="G$1" pin="ANODE"/>
+<wire x1="200.66" y1="-30.48" x2="200.66" y2="-33.02" width="0.1524" layer="91"/>
+</segment>
+</net>
+<net name="N$14" class="0">
+<segment>
+<pinref part="R15" gate="G$1" pin="P$1"/>
+<pinref part="D5" gate="G$1" pin="ANODE"/>
+<wire x1="208.28" y1="-30.48" x2="208.28" y2="-33.02" width="0.1524" layer="91"/>
+</segment>
+</net>

Commit message: power_dist r4: Checkpoint, most power/gnd routed
Connections:
- net N$3 renamed VIN_POST
Changed lines of the file:
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@@
 </segment>
 </net>
-<net name="N$3" class="0">
+<net name="VIN_POST" class="0">
 <segment>
 <wire x1="-33.02" y1="27.94" x2="-27.94" y2="27.94" width="0.1524" layer="91"/>

Commit message: power_dist r4: Routed and labels
Parts:
- added Q6: MF-DSC-SOT233-MMBT3904, mfdiscretesemi:NPN_BJTMMBT3904_SOT-23-3
Connections:
- new net N$3: Q6.BASE, Q6.COLLECTOR, U3.DIODE
- net CAN_SHDN: now also U2.PA15; no longer U2.PB14
- net GND: now also Q6.EMITTER
- net PWR_LED: now also U2.PB9; no longer U2.PA2
- net PWR_SW: now also U2.PB7; no longer U2.PA3
Changed lines of the file:
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@@
 </part>
 <part name="P+13" library="supply1" deviceset="VCC" device=""/>
+<part name="Q6" library="mfdiscretesemi" deviceset="NPN_BJT" device="_SOT-23-3" technology="MMBT3904" value="MF-DSC-SOT233-MMBT3904"/>
+<part name="GND25" library="supply1" deviceset="GND" device=""/>
 </parts>
 <sheets>
@@
 <attribute name="VALUE" x="205.74" y="-17.78" size="1.778" layer="96" rot="R90"/>
 </instance>
+<instance part="Q6" gate="G$1" x="63.5" y="-76.2" smashed="yes">
+<attribute name="NAME" x="68.58" y="-71.12" size="1.016" layer="95" font="vector" rot="R180" align="bottom-right"/>
+<attribute name="VALUE" x="68.58" y="-73.66" size="1.016" layer="96" font="vector"/>
+</instance>
+<instance part="GND25" gate="1" x="66.04" y="-88.9" smashed="yes">
+<attribute name="VALUE" x="63.5" y="-91.44" size="1.778" layer="96"/>
+</instance>
 </instances>
 <busses>
@@
 <pinref part="GND24" gate="1" pin="GND"/>
 <wire x1="269.24" y1="-53.34" x2="269.24" y2="-55.88" width="0.1524" layer="91"/>
+</segment>
+<segment>
+<pinref part="Q6" gate="G$1" pin="EMITTER"/>
+<pinref part="GND25" gate="1" pin="GND"/>
+<wire x1="66.04" y1="-83.82" x2="66.04" y2="-86.36" width="0.1524" layer="91"/>
 </segment>
 </net>
@@
 </segment>
 <segment>
-<pinref part="U2" gate="G$1" pin="PB14"/>
-<wire x1="492.76" y1="129.54" x2="525.78" y2="129.54" width="0.1524" layer="91"/>
-<label x="515.62" y="129.54" size="1.778" layer="95"/>
+<pinref part="U2" gate="G$1" pin="PA15"/>
+<wire x1="482.6" y1="175.26" x2="482.6" y2="190.5" width="0.1524" layer="91"/>
+<label x="482.6" y="182.88" size="1.778" layer="95" rot="R90"/>
 </segment>
 </net>
@@
 </segment>
 <segment>
-<pinref part="U2" gate="G$1" pin="PA3"/>
-<wire x1="447.04" y1="127" x2="421.64" y2="127" width="0.1524" layer="91"/>
-<label x="421.64" y="127" size="1.778" layer="95" font="vector"/>
+<pinref part="U2" gate="G$1" pin="PB7"/>
+<wire x1="464.82" y1="175.26" x2="464.82" y2="193.04" width="0.1524" layer="91"/>
+<label x="464.82" y="180.34" size="1.778" layer="95" rot="R90"/>
 </segment>
 </net>
@@
 </segment>
 <segment>
-<pinref part="U2" gate="G$1" pin="PA2"/>
-<wire x1="447.04" y1="129.54" x2="421.64" y2="129.54" width="0.1524" layer="91"/>
-<label x="421.64" y="129.54" size="1.778" layer="95" font="vector"/>
+<pinref part="U2" gate="G$1" pin="PB9"/>
+<wire x1="459.74" y1="175.26" x2="459.74" y2="193.04" width="0.1524" layer="91"/>
+<label x="459.74" y="180.34" size="1.778" layer="95" rot="R90"/>
 </segment>
 </net>
@@
 </segment>
 </net>
+<net name="N$3" class="0">
+<segment>
+<pinref part="U3" gate="A" pin="DIODE"/>
+<wire x1="40.64" y1="-53.34" x2="48.26" y2="-53.34" width="0.1524" layer="91"/>
+<wire x1="48.26" y1="-53.34" x2="48.26" y2="-55.88" width="0.1524" layer="91"/>
+<wire x1="48.26" y1="-55.88" x2="58.42" y2="-55.88" width="0.1524" layer="91"/>
+<wire x1="58.42" y1="-55.88" x2="58.42" y2="-66.04" width="0.1524" layer="91"/>
+<wire x1="58.42" y1="-66.04" x2="66.04" y2="-66.04" width="0.1524" layer="91"/>
+<pinref part="Q6" gate="G$1" pin="COLLECTOR"/>
+<wire x1="66.04" y1="-66.04" x2="66.04" y2="-68.58" width="0.1524" layer="91"/>
+<wire x1="58.42" y1="-66.04" x2="55.88" y2="-66.04" width="0.1524" layer="91"/>
+<junction x="58.42" y="-66.04"/>
+<pinref part="Q6" gate="G$1" pin="BASE"/>
+<wire x1="55.88" y1="-66.04" x2="55.88" y2="-76.2" width="0.1524" layer="91"/>
+</segment>
+</net>
