File: hw/power_dist/power_dist.sch (EAGLE design)
At the start: 69 parts, among them J1 JST-ZH6SMT_VERT, J2 JST-PH4SMT_VERT, J3 JST-PH5VERT, P1 XT30P, P2 XT30P, P3 XT30P, P4 XT30P, P5 XT30P, P6 XT30P, P7 XT90PW-M, Q1 PSMN4R8-100BSEJ, Q2 PSMN4R8-100BSEJ, Q3 PSMN4R8-100BSEJ, Q4 MF-DSC-SOT233-BSS138, Q5 MF-DSC-SOT233-MMBT3906, Q6 MF-DSC-SOT233-MMBT3904, U1 MAX15062AATA+T, U2 STM32G474CEU6, U3 LM5066IPMHE/NOPB, U4 TCAN334G

Commit message: power_dist r4: Update XT90 silk to be closer to actual part
Parts:
- P7: device precharge:XT90PW-M -> power_dist:XT90PW-M
Changed lines of the file:
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@@
 <attribute name="POPULATE" value="0"/>
 </part>
-<part name="P7" library="precharge" deviceset="XT90" device="PW-M">
+<part name="P7" library="power_dist" deviceset="XT90" device="PW-M">
 <attribute name="POPULATE" value="0"/>
 </part>
